Commit message: new pc
starting from new pc

File: hexapodo_description/robots/hexapodo.robot.xacro (robot description, xacro)
@@ -5,34 +5,34 @@
 <!--=====================================================================-->
 <!-- Archivos para incluir en el robot -->
-<xacro:include filename="$(find hexapodo_description)/urdf/pata_c.xacro"/>
-<xacro:include filename="$(find hexapodo_description)/urdf/base.xacro"/>
-<!--xacro:include filename="$(find hexapodo_description)/urdf/sensores/kinect_camera.xacro"/>
+<xacro:include filename="$(find hexapodo_description)/urdf/pata_c.robot.xacro"/>
+<xacro:include filename="$(find hexapodo_description)/urdf/base.robot.xacro"/>
+<xacro:include filename="$(find hexapodo_description)/urdf/sensores/kinect_camera.xacro"/>
 <xacro:include filename="$(find hexapodo_description)/urdf/sensores/imu.xacro"/>
-<xacro:include filename="$(find hexapodo_description)/urdf/sensores/hokuyo_sensor.xacro"/-->
+<xacro:include filename="$(find hexapodo_description)/urdf/sensores/hokuyo_sensor.xacro"/>
 <!-- Declaracion del plugin gazebo_ros_control -->
-<gazebo>
+<!--gazebo>
     <plugin name="gazebo_ros_control" filename="libgazebo_ros_control.so">
         <robotNamespace>/hexapodo</robotNamespace>
     </plugin>
-</gazebo>
+</gazebo-->
 <!-- Instanciacion de las patas dentro de la descripcion del robot -->
-<pata_c name="pata_1" parent_link="base_link" right="0">
+<motor name="motor_1" parent_link="base_link" right="0">
     <origin xyz="${-235/1000} ${233/1000} ${0/1000}" rpy="0 0 0"/>
-</pata_c>
-<pata_c name="pata_2" parent_link="base_link" right="1">
+</motor>
+<motor name="motor_2" parent_link="base_link" right="1">
     <origin xyz="${-235/1000} ${-233/1000} ${0/1000}" rpy="0 0 0"/>
-</pata_c>
-<pata_c name="pata_3" parent_link="base_link" right="0">
+</motor>
+<motor name="motor_3" parent_link="base_link" right="0">
     <origin xyz="${0/1000} ${289/1000} ${0/1000}" rpy="0 0 0"/>
-</pata_c>
-<pata_c name="pata_4" parent_link="base_link" right="1">
+</motor>
+<motor name="motor_4" parent_link="base_link" right="1">
     <origin xyz="${0/1000} ${-289/1000} ${0/1000}" rpy="0 0 0"/>
-</pata_c>
-<pata_c name="pata_5" parent_link="base_link" right="0">
+</motor>
+<motor name="motor_5" parent_link="base_link" right="0">
     <origin xyz="${235/1000} ${233/1000} ${0/1000}" rpy="0 0 0"/>
-</pata_c>
-<pata_c name="pata_6" parent_link="base_link" right="1">
+</motor>
+<motor name="motor_6" parent_link="base_link" right="1">
     <origin xyz="${235/1000} ${-233/1000} ${0/1000}" rpy="0 0 0"/>
-</pata_c>
+</motor>
 <!-- Instanciacion de la camara kinect dentro de la descripcion del robot -->
 <!--kinect_camera name="kin" parent_link="base_link">
@@ -40,9 +40,9 @@
 </kinect_camera-->
 <!-- Instanciacion de la IMU dentro de la descripcion del robot -->
-<!--imu name="imu1" parent_link="base_link">
+<imu name="imu1" parent_link="base_link">
     <origin xyz="${0/1000} ${0/1000} ${40/1000}" rpy="0 0 0"/>
-</imu-->
-<!--hokuyo_sensor sensor_name="hokuyo" parent_name="base_link">
+</imu>
+<hokuyo_sensor sensor_name="hokuyo" parent_name="base_link">
     <origin xyz="${300/1000} 0 0" rpy="0 0 0"/>
-</hokuyo_sensor-->
+</hokuyo_sensor>
 </robot>

File: hexapodo_description/robots/hexapodo_locked.xacro (robot description, xacro)
@@ -2,12 +2,12 @@
 <robot name="hexapodo" xmlns:xacro="http://ros.org/wiki/xacro">
 <!--=====================================================================-->
-<!--        Definicion del robot hexapodo                                    -->
+<!--        Definicion del robot hexapodo                                -->
 <!--=====================================================================-->
 <!-- Archivos para incluir en el robot -->
-<xacro:include filename="$(find hexapodo_description)/urdf/pata_c.xacro"/>
-<xacro:include filename="$(find hexapodo_description)/urdf/base.xacro"/>
-<!--xacro:include filename="$(find hexapodo_description)/urdf/sensores/kinect_camera.xacro"/>
-<xacro:include filename="$(find hexapodo_description)/urdf/sensores/imu.xacro"/>
-<xacro:include filename="$(find hexapodo_description)/urdf/sensores/hokuyo_sensor.xacro"/-->
+<xacro:include filename="$(find hexapodo_description)/urdf/pata_c_locked.xacro"/>
+<xacro:include filename="$(find hexapodo_description)/urdf/base_locked.xacro"/>
+<!--xacro:include filename="$(find hexapodo_description)/urdf/sensores/kinect_camera.xacro"/-->
+<!--xacro:include filename="$(find hexapodo_description)/urdf/sensores/imu.xacro"/-->
+<!--xacro:include filename="$(find hexapodo_description)/urdf/sensores/hokuyo_sensor.xacro"/-->
 <!-- Declaracion del plugin gazebo_ros_control -->
 <gazebo>

File: hexapodo_description/urdf/pata_c.robot.xacro (robot description, xacro)
@@ -1,10 +1,8 @@
 <?xml version="1.0" ?>
-<robot name="pata_c" xmlns:xacro="http://ros.org/wiki/xacro">
-<!--xacro:property name="motor_reduction"  value="${529.0/16}"/-->
-<xacro:property name="motor_reduction"  value="${1}"/>
-<!--xacro:property name="motor_max_effort" value="${3.5}"/-->
-<xacro:property name="motor_max_effort" value="${12}"/>
+<robot name="motor" xmlns:xacro="http://ros.org/wiki/xacro">
+<xacro:property name="motor_reduction"  value="${529.0/16}"/>
+<xacro:property name="motor_max_effort" value="${3.75}"/>
 <xacro:property name="motor_max_rev"    value="${1256.637/motor_reduction}"/>
-<xacro:macro name="pata_c" params="name parent_link right *origin">
+<xacro:macro name="motor" params="name parent_link right *origin">
     <!--=====================================================================-->
     <!--        Definicion de las patas en C del robot hexapodo              -->
@@ -13,5 +11,5 @@
     <!--Definicion del link de la pata-->
     <!--*******************************************************************************************-->
-    <link name="${name}_pata_c_link">
+    <link name="${name}_link">
         <!-- El origen de la pata varia en funcion de si se trata de una pata de la zona izquierda -->
         <!-- o de la zona derecha que se pasa como parametro -->
@@ -55,5 +53,5 @@
         <xacro:insert_block name="origin"/>
         <parent link="${parent_link}"/>
-        <child link="${name}_pata_c_link"/>
+        <child link="${name}_link"/>
         <axis xyz="0 1 0"/>
         <limit effort="${motor_max_effort}" velocity="${motor_max_rev}"/> <!-- Nm rads/s -->
@@ -65,9 +63,9 @@
         <type>transmission_interface/SimpleTransmission</type>
         <joint name="${name}_to_${parent_link}_joint">
-            <hardwareInterface>hardware_interface/EffortJointInterface</hardwareInterface>
+            <hardwareInterface>hardware_interface/VelocityJointInterface</hardwareInterface>
         </joint>
-        <actuator name="${name}_motor">
+        <actuator name="hexapodo/${name}_actuator">
             <mechanicalReduction>${motor_reduction}</mechanicalReduction>
-            <hardwareInterface>EffortJointInterface</hardwareInterface>
+            <hardwareInterface>hardware_interface/VelocityJointInterface</hardwareInterface>
         </actuator>
     </transmission>
@@ -75,9 +73,9 @@
     <!--Definicion de las propiedades de gazebo-->
     <!--*******************************************************************************************-->
-    <gazebo reference="${name}_pata_c_link">
-        <mu1>100000.0</mu1>
-        <mu2>100000.0</mu2>
+    <!--<gazebo reference="${name}_link">
+        <mu1>1</mu1>
+        <mu2>1</mu2>
         <material>Gazebo/Grey</material>
-    </gazebo>
+    </gazebo-->
 </xacro:macro>
 </robot>

File: hexapodo_description/urdf/pata_c_locked.xacro (robot description, xacro)
@@ -1,8 +1,6 @@
 <?xml version="1.0" ?>
 <robot name="pata_c" xmlns:xacro="http://ros.org/wiki/xacro">
-<!--xacro:property name="motor_reduction"  value="${529.0/16}"/-->
-<xacro:property name="motor_reduction"  value="${1}"/>
-<!--xacro:property name="motor_max_effort" value="${3.5}"/-->
-<xacro:property name="motor_max_effort" value="${12}"/>
+<xacro:property name="motor_reduction"  value="${529.0/16}"/>
+<xacro:property name="motor_max_effort" value="${3.75}"/>
 <xacro:property name="motor_max_rev"    value="${1256.637/motor_reduction}"/>
 <xacro:macro name="pata_c" params="name parent_link right *origin">
@@ -13,5 +11,5 @@
     <!--Definicion del link de la pata-->
     <!--*******************************************************************************************-->
-    <link name="${name}_pata_c_link">
+    <link name="${name}_link">
         <!-- El origen de la pata varia en funcion de si se trata de una pata de la zona izquierda -->
         <!-- o de la zona derecha que se pasa como parametro -->
@@ -55,5 +53,5 @@
         <xacro:insert_block name="origin"/>
         <parent link="${parent_link}"/>
-        <child link="${name}_pata_c_link"/>
+        <child link="${name}_link"/>
         <axis xyz="0 1 0"/>
         <limit effort="${motor_max_effort}" velocity="${motor_max_rev}"/> <!-- Nm rads/s -->
@@ -67,5 +65,5 @@
             <hardwareInterface>hardware_interface/EffortJointInterface</hardwareInterface>
         </joint>
-        <actuator name="${name}_motor">
+        <actuator name="${name}_actuator">
             <mechanicalReduction>${motor_reduction}</mechanicalReduction>
             <hardwareInterface>EffortJointInterface</hardwareInterface>
@@ -75,7 +73,7 @@
     <!--Definicion de las propiedades de gazebo-->
     <!--*******************************************************************************************-->
-    <gazebo reference="${name}_pata_c_link">
-        <mu1>100000.0</mu1>
-        <mu2>100000.0</mu2>
+    <gazebo reference="${name}_link">
+        <mu1>1</mu1>
+        <mu2>1</mu2>
         <material>Gazebo/Grey</material>
     </gazebo>
