Commit message: Probando el tripode alterno pose
Proando el tripode alterno pose, se cae al probar el segundo tripoe, luego se recupera.

File: hexapodo_description/urdf/pata_c.xacro (robot description, xacro)
@@ -3,6 +3,6 @@
 <!--xacro:property name="motor_reduction"  value="${529.0/16}"/-->
 <xacro:property name="motor_reduction"  value="${1}"/>
-<!--xacro:property name="motor_max_effort" value="${3.5}"/-->
-<xacro:property name="motor_max_effort" value="${12}"/>
+<xacro:property name="motor_max_effort" value="${3.5}"/>
+<!--xacro:property name="motor_max_effort" value="${12}"/-->
 <xacro:property name="motor_max_rev"    value="${1256.637/motor_reduction}"/>
 <xacro:macro name="pata_c" params="name parent_link right *origin">
@@ -47,4 +47,14 @@
                 <mesh filename="package://hexapodo_description/meshes/pvc.stl" scale="0.001 0.001 0.001"/>
             </geometry>
+            <surface>
+              <friction>
+                <ode>
+                  <mu>100000.0</mu>
+                  <mu2>100000.0</mu2>
+                  <slip1>0.0</slip1>
+                  <slip2>0.0</slip2>
+                </ode>
+              </friction>
+            </surface>
         </collision>
     </link>
@@ -76,6 +86,9 @@
     <!--*******************************************************************************************-->
     <gazebo reference="${name}_pata_c_link">
-        <mu1>100000.0</mu1>
-        <mu2>100000.0</mu2>
+        <mu1 value="100000.0"/>
+        <mu2 value="100000.0"/>
+        <kp  value="10000000.0" />
+        <kd  value="1.0" />
+        <fdir1 value="1 0 0"/>
         <material>Gazebo/Grey</material>
     </gazebo>
